File: pcb/CC40_RAM_Cart.brd (EAGLE design)
At the start: 43.2 x 48 mm, 16 parts, among them IC2 AS6CX008, X1 EXPANSION_PORT_CC40_EDGE

Commit message: Updated layouts and measurements
Parts:
- added P1: CC40_CARTN, ti-cc40-74-95:CC40_CART_NOHOLE
- S1: device switch-dil:DP-04 -> switch-dil-rp:DP-04
- X1: value EXPANSION_PORT_CC40_EDGE -> EXPANSION_PORT_CC40; device ti-cc40:MA20-2(.050) -> ti-cc40-74-95:MA20-2(.050)
- moved X1 1.27 mm to (0.00, 5.08)
Routing:
- net A9: track 22.8 -> 21.7 mm
- net VCC: track 65.7 -> 64.8 mm
- net A14: track 36.9 -> 36.0 mm
- net P25.2: track 54.5 -> 53.5 mm
- net N$7: track 36.7 -> 35.7 mm
- net A6: track 32.7 -> 31.7 mm
- net A5: track 33.2 -> 32.2 mm
- net A4: track 33.7 -> 32.7 mm
- net A3: track 34.2 -> 33.3 mm
- net A2: track 35.3 -> 34.3 mm
- net A12: track 33.2 -> 32.2 mm
- net A8: track 30.1 -> 29.1 mm
- net A11: track 21.0 -> 20.1 mm
- net A10: track 17.4 -> 16.4 mm
- net P25.3: track 33.4 -> 32.4 mm
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Other:
- outline, holes or cut-outs redrawn
