File: pcb/CC40_RAM_Cart.sch (EAGLE design)
At the start: 16 parts, among them IC2 AS6CX008, X1 EXPANSION_PORT_CC40_EDGE

Commit message: Updated layouts and measurements
Parts:
- added P1: CC40_CARTN, ti-cc40-74-95:CC40_CARTN
- S1: device switch-dil:DP04 -> switch-dil-rp:DP04
- X1: value EXPANSION_PORT_CC40_EDGE -> EXPANSION_PORT_CC40; device ti-cc40:EXPANSION_PORT_CC40_EDGE -> ti-cc40-74-95:EXPANSION_PORT_CC40
Connections:
- net !OE: now also IC2A.!OE; no longer IC2G$1.!OE
- net !WE: now also IC2A.!WE; no longer IC2G$1.!WE
- net A0: now also IC2A.A0; no longer IC2G$1.A0
- net A1: now also IC2A.A1; no longer IC2G$1.A1
- net A10: now also IC2A.A10; no longer IC2G$1.A10
- net A11: now also IC2A.A11; no longer IC2G$1.A11
- net A12: now also IC2A.A12; no longer IC2G$1.A12
- net A13: now also IC2A.A13; no longer IC2G$1.A13
- net A14: now also IC2A.A14; no longer IC2G$1.A14
- net A2: now also IC2A.A2; no longer IC2G$1.A2
- net A3: now also IC2A.A3; no longer IC2G$1.A3
- net A4: now also IC2A.A4; no longer IC2G$1.A4
- net A5: now also IC2A.A5; no longer IC2G$1.A5
- net A6: now also IC2A.A6; no longer IC2G$1.A6
- net A7: now also IC2A.A7; no longer IC2G$1.A7
- net A8: now also IC2A.A8; no longer IC2G$1.A8
- net A9: now also IC2A.A9; no longer IC2G$1.A9
- net D0: now also IC2A.D0; no longer IC2G$1.D0
- net D1: now also IC2A.D1; no longer IC2G$1.D1
- net D2: now also IC2A.D2; no longer IC2G$1.D2
- net D3: now also IC2A.D3; no longer IC2G$1.D3
- net D4: now also IC2A.D4; no longer IC2G$1.D4
- net D5: now also IC2A.D5; no longer IC2G$1.D5
- net D6: now also IC2A.D6; no longer IC2G$1.D6
- net D7: now also IC2A.D7; no longer IC2G$1.D7
- net N$1: now also IC2A.!CE, X1X.!CS_RAM, X1X.!CS_ROM; no longer IC2G$1.!CE, X1X.!CS_CRAM, X1X.!CS_CROM
- net SA15: now also IC2A.A15; no longer IC2G$1.A15
- net SA16: now also IC2A.A16; no longer IC2G$1.A16
- net SA17: now also IC2A.A17; no longer IC2G$1.A17
- net SA18: now also IC2A.A18; no longer IC2G$1.A18
